File: emb/project/punbox/hw/punbox.kicad_pcb (KiCad board)
At the start: 2 copper layers, 50 x 75 mm, 12 parts, among them J2 Speakers, J3 Button, U1 MAX98357A, U2 MAX98357A

Commit message: better routing, 3d model fixes
Parts:
- moved J3 46.4 mm to (122.0, 72.0)
- moved C1 18.6 mm to (115.6, 88.0)
- moved C3 18.6 mm to (115.4, 86.0)
- moved C4 18.6 mm to (127.4, 86.0)
- moved R1 18.6 mm to (117.5, 82.5)
- moved R2 18.6 mm to (129.5, 82.5)
- moved C2 18.6 mm to (127.6, 88.0)
- moved J2 18.6 mm to (123.4, 94.5)
- moved U1 18.6 mm to (119.3, 87.2)
- moved U2 18.6 mm to (131.3, 87.2)
Routing:
- net +5V: track 0.00 -> 93.0 mm
- net I2S_LRCLK: track 0.00 -> 58.2 mm, vias 0 -> 3
- net I2S_BCLK: track 0.00 -> 47.5 mm, vias 0 -> 3
- net I2S_DIN: track 0.00 -> 42.3 mm, vias 0 -> 3
- net BUTTON: track 0.00 -> 38.3 mm
- net GND: track 0.00 -> 17.9 mm, vias 0 -> 11
- net N$3: track 0.00 -> 8.76 mm
- net N$4: track 0.00 -> 7.88 mm
- net N$2: track 0.00 -> 6.12 mm
- net N$1: track 0.00 -> 5.81 mm
- net U2_SD_MODE: track 0.00 -> 3.39 mm
- net U1_SD_MODE: track 0.00 -> 3.39 mm
- added copper zone on B.Cu, net GND
Other:
- board size 50 x 75 mm -> 55 x 55 mm

Commit message: final v1 design
Parts:
- added REF**: MountingHole_2.7mm_M2.5, MountingHole:MountingHole_2.7mm_M2.5, F.Cu at (127.0, 48.5)
- added REF**: MountingHole_2.7mm_M2.5, MountingHole:MountingHole_2.7mm_M2.5, F.Cu at (127.0, 97.0)
- added REF**: MountingHole_2.7mm_M2.5, MountingHole:MountingHole_2.7mm_M2.5, F.Cu at (80.0, 97.0)
- added REF**: MountingHole_2.7mm_M2.5, MountingHole:MountingHole_2.7mm_M2.5, F.Cu at (80.0, 48.5)
- J3: footprint punbox_parts:JST_PH_B2B-PH-K_1x02_P2.00mm_Vertical -> punbox_parts:JST_XH_B2B-XH-A_1x02_P2.50mm_Vertical
- moved R2 7.53 mm to (122.0, 82.5)
- moved C4 7.35 mm to (120.0, 86.0)
- moved C2 7.35 mm to (120.3, 88.0)
- moved U2 7.29 mm to (124.0, 87.2)
- moved J2 5.42 mm to (118.0, 94.5)
- moved U1 4.04 mm to (115.2, 87.2)
- moved R1 4.03 mm to (113.5, 82.5)
- moved C1 3.95 mm to (111.6, 88.0)
- moved C3 3.95 mm to (111.5, 86.0)
- moved J3 3.65 mm to (118.5, 73.0)
- moved C5 3.00 mm to (115.0, 51.0)
Routing:
- net +5V: track 93.0 -> 83.9 mm
- net I2S_DIN: track 42.3 -> 37.9 mm
- net I2S_LRCLK: track 58.2 -> 54.3 mm
- net I2S_BCLK: track 47.5 -> 44.2 mm
- net N$3: track 8.76 -> 8.09 mm
- net BUTTON: track 38.3 -> 37.7 mm
- net N$1: track 5.81 -> 5.24 mm
Other:
- board size 55 x 55 mm -> 53 x 54.5 mm
- board text added: "Punbox V1 - Ryan"
